Commit message: Increase default height of lift joint

File: resource/urdf/stretch/stretch.urdf (robot description, URDF)
Before this commit: robot stretch, 20 links, 19 joints
Joints:
- joint joint_lift: origin xyz=-0.037385 0.1666 0 rpy=-1.5708 1.5708 0 -> xyz=-0.037385 0.3666 0 rpy=-1.5708 1.5708 0
