Commit message: changed finger collision & friction

File: resource/urdf/robot/robot.urdf (robot description, URDF)
Before this commit: robot robot, 24 links, 23 joints
Links:
- link left_link_finger: geometry collision box size=0.01 0.03 0.03; visual box size=0.01 0.03 0.03

Commit message: changed gripper width

File: resource/urdf/robot/robot.urdf (robot description, URDF)
Before this commit: robot robot, 24 links, 23 joints
Links:
- link left_link_finger: geometry collision box size=0.005 0.03 0.03; visual box size=0.005 0.03 0.03
- link link_gripper: geometry collision box size=0.08 0.03 0.03; visual box size=0.08 0.03 0.03
- link right_link_finger: geometry collision box size=0.005 0.03 0.03; visual box size=0.005 0.03 0.03
Joints:
- joint joint_left_finger: limit lower=-0.03 upper=0.02 effort=100 velocity=1.0 -> lower=-0.03 upper=0.005 effort=100 velocity=1.0
- joint joint_right_finger: limit lower=-0.02 upper=0.03 effort=100 velocity=1.0 -> lower=-0.005 upper=0.03 effort=100 velocity=1.0

Commit message: optimized gripper
- ensured the robot arm is can reach far enough
- made sure the chess piece does not move around when gripped (better friction on gripper)
- set the highest and lowest point the robot arm can move such that it will not hit the table

File: resource/urdf/robot/robot.urdf (robot description, URDF)
Before this commit: robot robot, 24 links, 23 joints
Joints:
- joint joint_arm_l0: limit lower=0.0 upper=0.13 effort=100 velocity=1.0 -> lower=0.0 upper=0.15 effort=100 velocity=1.0
- joint joint_arm_l1: limit lower=0.0 upper=0.13 effort=100 velocity=1.0 -> lower=0.0 upper=0.2 effort=100 velocity=1.0
- joint joint_arm_l2: limit lower=0.0 upper=0.13 effort=100 velocity=1.0 -> lower=0.0 upper=0.2 effort=100 velocity=1.0
- joint joint_arm_l3: limit lower=0.0 upper=0.13 effort=100 velocity=1.0 -> lower=0.0 upper=0.2 effort=100 velocity=1.0
- joint joint_lift: limit lower=0.0 upper=1.1 effort=100 velocity=1.0 -> lower=-0.01 upper=0.0 effort=100 velocity=2.0; origin xyz=-0.037385 0.3666 0 rpy=-1.5708 1.5708 0 -> xyz=-0.037385 0.7 0 rpy=-1.5708 1.5708 0

Commit message: added indexes

File: resource/urdf/robot/robot.urdf (robot description, URDF)
Before this commit: robot robot, 24 links, 23 joints
Joints:
- joint joint_lift: limit lower=-0.01 upper=0.0 effort=100 velocity=2.0 -> lower=-0.015 upper=0.0 effort=100 velocity=2.0; origin xyz=-0.037385 0.7 0 rpy=-1.5708 1.5708 0 -> xyz=-0.037385 0.705 0 rpy=-1.5708 1.5708 0
