Commit message: added mass and inertia

File: resource/urdf/obj_libs/chessboard/chessboard.urdf (robot description, URDF)
Before this commit: robot chessboard.urdf, 1 links, 0 joints
Links:
- link chessboard: mass None -> 0.01

File: resource/urdf/obj_libs/chesspieces/b1/model.urdf (robot description, URDF)
Before this commit: robot chesspiece1.urdf, 1 links, 0 joints
Links:
- link chesspiece1: mass None -> 0.01

File: resource/urdf/obj_libs/chesspieces/b10/model.urdf (robot description, URDF)
Before this commit: robot chesspiece10.urdf, 1 links, 0 joints
Links:
- link chesspiece10: mass None -> 0.01

File: resource/urdf/obj_libs/chesspieces/b11/model.urdf (robot description, URDF)
Before this commit: robot chesspiece11.urdf, 1 links, 0 joints
Links:
- link chesspiece11: mass None -> 0.01

File: resource/urdf/obj_libs/chesspieces/b12/model.urdf (robot description, URDF)
Before this commit: robot chesspiece12.urdf, 1 links, 0 joints
Links:
- link chesspiece12: mass None -> 0.01

File: resource/urdf/obj_libs/chesspieces/b13/model.urdf (robot description, URDF)
Before this commit: robot chesspiece13.urdf, 1 links, 0 joints
Links:
- link chesspiece13: mass None -> 0.01

File: resource/urdf/obj_libs/chesspieces/b14/model.urdf (robot description, URDF)
Before this commit: robot chesspiece14.urdf, 1 links, 0 joints
Links:
- link chesspiece14: mass None -> 0.01

File: resource/urdf/obj_libs/chesspieces/b15/model.urdf (robot description, URDF)
Before this commit: robot chesspiece15.urdf, 1 links, 0 joints
Links:
- link chesspiece15: mass None -> 0.01

File: resource/urdf/obj_libs/chesspieces/b16/model.urdf (robot description, URDF)
Before this commit: robot chesspiece16.urdf, 1 links, 0 joints
Links:
- link chesspiece16: mass None -> 0.01

File: resource/urdf/obj_libs/chesspieces/b2/model.urdf (robot description, URDF)
Before this commit: robot chesspiece2.urdf, 1 links, 0 joints
Links:
- link chesspiece2: mass None -> 0.01

File: resource/urdf/obj_libs/chesspieces/b3/model.urdf (robot description, URDF)
Before this commit: robot chesspiece3.urdf, 1 links, 0 joints
Links:
- link chesspiece3: mass None -> 0.01

File: resource/urdf/obj_libs/chesspieces/b4/model.urdf (robot description, URDF)
Before this commit: robot chesspiece4.urdf, 1 links, 0 joints
Links:
- link chesspiece4: mass None -> 0.01

File: resource/urdf/obj_libs/chesspieces/b5/model.urdf (robot description, URDF)
Before this commit: robot chesspiece5.urdf, 1 links, 0 joints
Links:
- link chesspiece5: mass None -> 0.01

File: resource/urdf/obj_libs/chesspieces/b6/model.urdf (robot description, URDF)
Before this commit: robot chesspiece6.urdf, 1 links, 0 joints
Links:
- link chesspiece6: mass None -> 0.01

File: resource/urdf/obj_libs/chesspieces/b7/model.urdf (robot description, URDF)
Before this commit: robot chesspiece7.urdf, 1 links, 0 joints
Links:
- link chesspiece7: mass None -> 0.01

File: resource/urdf/obj_libs/chesspieces/b8/model.urdf (robot description, URDF)
Before this commit: robot chesspiece8.urdf, 1 links, 0 joints
Links:
- link chesspiece8: mass None -> 0.01

File: resource/urdf/obj_libs/chesspieces/b9/model.urdf (robot description, URDF)
Before this commit: robot chesspiece9.urdf, 1 links, 0 joints
Links:
- link chesspiece9: mass None -> 0.01

File: resource/urdf/obj_libs/chesspieces/r1/model.urdf (robot description, URDF)
Before this commit: robot chesspiece17.urdf, 1 links, 0 joints
Links:
- link chesspiece17: mass None -> 0.01

File: resource/urdf/obj_libs/chesspieces/r10/model.urdf (robot description, URDF)
Before this commit: robot chesspiece26.urdf, 1 links, 0 joints
Links:
- link chesspiece26: mass None -> 0.01

File: resource/urdf/obj_libs/chesspieces/r11/model.urdf (robot description, URDF)
Before this commit: robot chesspiece27.urdf, 1 links, 0 joints
Links:
- link chesspiece27: mass None -> 0.01
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