Commit message: flipped chessboard img added box

File: resource/urdf/obj_libs/box/box.urdf (robot description, URDF)
Before this commit: robot chessboard.urdf, 1 links, 0 joints
Links:
- removed link chessboard
- added link box, mass 0.01; collision mesh filename=box.obj; visual mesh filename=box.obj
