Commit message: scaled the table

File: resource/urdf/table.urdf (robot description, URDF)
Before this commit: robot table.urdf, 1 links, 0 joints
Links:
- link baseLink: geometry collision box size=1.5 1 0.05; visual mesh filename=table.obj scale=0.1 0.1 0.58

Commit message: updated table collision

File: resource/urdf/table.urdf (robot description, URDF)
Before this commit: robot table.urdf, 1 links, 0 joints
Links:
- link baseLink: geometry collision box size=1.5 1.2 0.05; visual mesh filename=table.obj scale=0.1 0.1 0.58
